File: DH-DOM-0/DH-DOM-0_LSM6DSOXTR.kicad_pcb (KiCad board)
At the start: 2 copper layers, 40 x 40 mm, 45 parts, among them J1 USB_C_Receptacle_USB2.0_14P, J2 Conn_01x02, Q1 FDN340P, SW1 RST, SW2 BOOT, U2 MMC5983MA, U4 NCP1117-3.3_SOT223, U5 TVS1400DRV, U6 ESP32-S3-WROOM-1-N4R8, U7 TP4057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

Commit message: edit
separate versions for different IMUs, same footprint but traces have miniscule differences.
Parts:
- removed U9: LSM6DSV16BTR, Package_LGA:LGA-14_3x2.5mm_P0.5mm_LayoutBorder3x4y
- added U1: LSM6DSOXTR, footprints:LGA-14L_STM-M, F.Cu at (148.0, 106.5)
Routing:
- net GND: track 19.4 -> 12.1 mm, vias 2 -> 1
