File: DH-DOM-0/DH-DOM-0.kicad_sch (KiCad schematic)
At the start: 45 parts, among them J1 USB_C_Receptacle_USB2.0_14P, J2 Conn_01x02, Q1 FDN340P, SW1 RST, SW2 BOOT, U1 LSM6DSV16BTR, U2 LSM6DSOXTR, U3 MMC5983MA, U4 BMI270, U5 NCP1117-3.3_SOT223, U6 TVS1400DRV, U7 ESP32-S3-WROOM-1-N4R8, U8 TP4057, U9 ST7789

Commit message: edit
dont know either
Parts:
- BTN2, BTN3, BTN4: footprint Connector_PinHeader_2.00mm:PinHeader_2x01_P2.00mm_Vertical -> Connector_PinHeader_2.00mm:PinHeader_2x01_P2.00mm_Horizontal
Connections:
- net +3V3: now also BTN1.2, BTN2.2, BTN3.2, BTN4.2; no longer BTN1.1, BTN2.1, BTN3.1, BTN4.1
- net BTN1: now also BTN1.1; no longer BTN1.2
- net BTN2: now also BTN2.1; no longer BTN2.2
- net BTN3: now also BTN3.1; no longer BTN3.2
- net BTN4: now also BTN4.1; no longer BTN4.2
Other:
- moved on the sheet: BTN1, BTN2, BTN3, BTN4
Changed lines of the file:
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@@
 	(symbol
 		(lib_id "Switch:SW_Push")
-		(at 33.02 128.27 0)
+		(at 33.02 128.27 180)
 		(unit 1)
 		(body_style 1)
@@
 		(dnp no)
 		(property "Reference" "BTN2"
-			(at 35.814 125.984 0)
+			(at 30.226 130.556 0)
 			(show_name no)
 			(do_not_autoplace no)
@@
 		)
 		(property "Value" "SW_Push"
-			(at 33.02 123.19 0)
-			(hide yes)
-			(show_name no)
-			(do_not_autoplace no)
-			(effects
-				(font
-					(size 1.27 1.27)
-				)
-			)
-		)
-		(property "Footprint" "Connector_PinHeader_2.00mm:PinHeader_2x01_P2.00mm_Vertical"
-			(at 33.02 123.19 0)
-			(hide yes)
-			(show_name no)
-			(do_not_autoplace no)
-			(effects
-				(font
-					(size 1.27 1.27)
-				)
-			)
-		)
-		(property "Datasheet" ""
-			(at 33.02 123.19 0)
+			(at 33.02 133.35 0)
+			(hide yes)
+			(show_name no)
+			(do_not_autoplace no)
+			(effects
+				(font
+					(size 1.27 1.27)
+				)
+			)
+		)
+		(property "Footprint" "Connector_PinHeader_2.00mm:PinHeader_2x01_P2.00mm_Horizontal"
+			(at 33.02 133.35 0)
+			(hide yes)
+			(show_name no)
+			(do_not_autoplace no)
+			(effects
+				(font
+					(size 1.27 1.27)
+				)
+			)
+		)
+		(property "Datasheet" ""
+			(at 33.02 133.35 0)
 			(hide yes)
 			(show_name no)
@@
 	(symbol
 		(lib_id "Switch:SW_Push")
-		(at 33.02 138.43 0)
+		(at 33.02 138.43 180)
 		(unit 1)
 		(body_style 1)
@@
 		(dnp no)
 		(property "Reference" "BTN4"
-			(at 35.814 136.144 0)
+			(at 30.226 140.716 0)
 			(show_name no)
 			(do_not_autoplace no)
@@
 		)
 		(property "Value" "SW_Push"
-			(at 33.02 133.35 0)
-			(hide yes)
-			(show_name no)
-			(do_not_autoplace no)
-			(effects
-				(font
-					(size 1.27 1.27)
-				)
-			)
-		)
-		(property "Footprint" "Connector_PinHeader_2.00mm:PinHeader_2x01_P2.00mm_Vertical"
-			(at 33.02 133.35 0)
-			(hide yes)
-			(show_name no)
-			(do_not_autoplace no)
-			(effects
-				(font
-					(size 1.27 1.27)
-				)
-			)
-		)
-		(property "Datasheet" ""
-			(at 33.02 133.35 0)
+			(at 33.02 143.51 0)
+			(hide yes)
+			(show_name no)
+			(do_not_autoplace no)
+			(effects
+				(font
+					(size 1.27 1.27)
+				)
+			)
+		)
+		(property "Footprint" "Connector_PinHeader_2.00mm:PinHeader_2x01_P2.00mm_Horizontal"
+			(at 33.02 143.51 0)
+			(hide yes)
+			(show_name no)
+			(do_not_autoplace no)
+			(effects
+				(font
+					(size 1.27 1.27)
+				)
+			)
+		)
+		(property "Datasheet" ""
+			(at 33.02 143.51 0)
 			(hide yes)
 			(show_name no)
@@
 	(symbol
 		(lib_id "Switch:SW_Push")
-		(at 33.02 123.19 0)
+		(at 33.02 123.19 180)
 		(unit 1)
 		(body_style 1)
@@
 		(dnp no)
 		(property "Reference" "BTN1"
-			(at 35.814 120.904 0)
+			(at 30.226 125.476 0)
 			(show_name no)
 			(do_not_autoplace no)
@@
 		)
 		(property "Value" "SW_Push"
-			(at 33.02 118.11 0)
+			(at 33.02 128.27 0)
 			(hide yes)
 			(show_name no)
@@
 		)
 		(property "Footprint" "Connector_PinHeader_2.00mm:PinHeader_2x01_P2.00mm_Horizontal"
-			(at 33.02 118.11 0)
-			(hide yes)
-			(show_name no)
-			(do_not_autoplace no)
-			(effects
-				(font
-					(size 1.27 1.27)
-				)
-			)
-		)
-		(property "Datasheet" ""
-			(at 33.02 118.11 0)
+			(at 33.02 128.27 0)
+			(hide yes)
+			(show_name no)
+			(do_not_autoplace no)
+			(effects
+				(font
+					(size 1.27 1.27)
+				)
+			)
+		)
+		(property "Datasheet" ""
+			(at 33.02 128.27 0)
 			(hide yes)
 			(show_name no)
@@
 	(symbol
 		(lib_id "Switch:SW_Push")
-		(at 33.02 133.35 0)
+		(at 33.02 133.35 180)
 		(unit 1)
 		(body_style 1)
@@
 		(dnp no)
 		(property "Reference" "BTN3"
-			(at 35.814 131.064 0)
+			(at 30.226 135.636 0)
 			(show_name no)
 			(do_not_autoplace no)
@@
 		)
 		(property "Value" "SW_Push"
-			(at 33.02 128.27 0)
-			(hide yes)
-			(show_name no)
-			(do_not_autoplace no)
-			(effects
-				(font
-					(size 1.27 1.27)
-				)
-			)
-		)
-		(property "Footprint" "Connector_PinHeader_2.00mm:PinHeader_2x01_P2.00mm_Vertical"
-			(at 33.02 128.27 0)
-			(hide yes)
-			(show_name no)
-			(do_not_autoplace no)
-			(effects
-				(font
-					(size 1.27 1.27)
-				)
-			)
-		)
-		(property "Datasheet" ""
-			(at 33.02 128.27 0)
-			(hide yes)
-			(show_name no)
+			(at 33.02 138.43 0)
+			(hide yes)
+			(show_name no)
+			(do_not_autoplace no)
+			(effects
+				(font
+					(size 1.27 1.27)
+				)
+			)
+		)
+		(property "Footprint" "Connector_PinHeader_2.00mm:PinHeader_2x01_P2.00mm_Horizontal"
+			(at 33.02 138.43 0)
+			(hide yes)
+			(show_name no)
+			(do_not_autoplace no)
+			(effects
+				(font
+					(size 1.27 1.27)
+				)
+			)
+		)
+		(property "Datasheet" ""
+			(at 33.02 138.43 0)
+			(hide yes)
+			(show_name no)

Commit message: eduiyuyt
durrrrrrrr
Parts:
- U1, U2: now left out of the parts list
- renumbered C15 to C14, C14 to C15
Other:
- moved on the sheet: C5, C6, C7, C8, R1, R2, SW1, SW2, U5, U7
