File: DH-DOM-0/BMI270 VERSION/DH-DOM-0_BMI270.kicad_pcb (KiCad board)
At the start: 2 copper layers, 40 x 40 mm, 45 parts, among them J1 USB_C_Receptacle_USB2.0_14P, J2 Conn_01x02, Q1 FDN340P, SW1 RST, SW2 BOOT, U2 MMC5983MA, U3 BMI270, U4 NCP1117-3.3_SOT223, U5 TVS1400DRV, U6 ESP32-S3-WROOM-1-N4R8, U7 TP4057, U8 ST7789

Commit message: eduiyuyt
durrrrrrrr
Parts:
- removed the U3 at (148.0, 106.5)
- added C15: 100n, Capacitor_SMD:C_0805_2012Metric, F.Cu at (144.7, 115.0)
- added C3: 100n, Capacitor_SMD:C_0805_2012Metric, F.Cu at (141.6, 102.0)
- added U4: BMI270, Package_LGA:Bosch_LGA-14_3x2.5mm_P0.5mm, F.Cu at (148.0, 106.6)
- BTN1, BTN2, BTN3, BTN4: footprint Connector_PinHeader_2.54mm:PinHeader_2x01_P2.54mm_Vertical -> Connector_PinHeader_2.00mm:PinHeader_2x01_P2.00mm_Horizontal
- J2: footprint Connector_PinHeader_2.54mm:PinHeader_2x01_P2.54mm_Vertical -> Connector_PinHeader_2.00mm:PinHeader_2x01_P2.00mm_Vertical
- moved R3 2.48 mm to (139.4, 100.0), turned to -90 degrees
- moved R4 2.36 mm to (139.5, 103.4), turned to -90 degrees
- moved BTN4 2.03 mm to (166.4, 87.7), turned to 0 degrees
- moved BTN3 2.00 mm to (166.4, 91.3), turned to 0 degrees
- moved BTN1 2.00 mm to (166.4, 98.5), turned to 0 degrees
- moved BTN2 2.00 mm to (166.4, 94.9), turned to 0 degrees
- renumbered C9 to C10, C10 to C11, C11 to C12, C12 to C13, C13 to C14, C3 to C4, C4 to C5, C5 to C6, C6 to C7, C7 to C8, C8 to C9, U2 to U3, U4 to U5, U5 to U6, U6 to U7, U7 to U8, U8 to U9
Connections:
- BTN1 pad 1: +3V3 -> /BTN1
- BTN1 pad 2: /BTN1 -> +3V3
- BTN2 pad 1: +3V3 -> /BTN2
- BTN2 pad 2: /BTN2 -> +3V3
- BTN3 pad 1: +3V3 -> /BTN3
- BTN3 pad 2: /BTN3 -> +3V3
- BTN4 pad 1: +3V3 -> /BTN4
- BTN4 pad 2: /BTN4 -> +3V3
Routing:
- net +3V3: track 134.0 -> 142.4 mm, vias 8 -> 10
- net Net-(J1-CC1): track 6.64 -> 4.23 mm
- net GND: track 11.9 -> 13.4 mm
- net /BTN1: track 13.2 -> 11.8 mm
